File: HierarchyTest.kicad_sch (KiCad schematic)
At the start: 1 part, among them U1 4555

Commit message: updates
Parts:
- added unit 2 of U1
- added U2: 4555, symbol 4xxx_IEEE:4555
- added U3: 74AHC04, symbol 74xx:74AHC04
Other:
- added sheet Acc (accessory.kicad_sch)
