File: HierarchyTest.kicad_sch (KiCad schematic)
At the start: 3 parts, among them U1 4555, U2 4555, U3 74AHC04

Commit message: more updates
Other:
- added sheet BidirPins (PinsBidir.kicad_sch)
- added sheet InPins (PinsIn.kicad_sch)
- added sheet OutPins (PinsOut.kicad_sch)
- added sheet PassivePins (PinsPassive.kicad_sch)
- added sheet TriPins (PinsTri.kicad_sch)
Changed lines of the file:
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@@
   )
   (text "HIERARCHY IS ANARCHY" (at 54.61 21.59 0)
-    (effects (font (size 1.27 1.27)) (justify left bottom))
+    (effects (font (size 1.27 1.27) (color 255 18 90 0.8)) (justify left bottom))
   )
   (symbol (lib_id "4xxx_IEEE:4555") (at 113.665 54.61 0) (unit 2)
@@
           (reference "U3") (unit 3)
         )
+      )
+    )
+  )
+  (sheet (at 39.37 124.46) (size 23.495 19.05) (fields_autoplaced)
+    (stroke (width 0.1524) (type solid))
+    (fill (color 0 0 0 0.0000))
+    (property "Sheetname" "OutPins" (at 39.37 123.7484 0)
+      (effects (font (size 1.27 1.27)) (justify left bottom))
+    )
+    (property "Sheetfile" "PinsOut.kicad_sch" (at 39.37 144.0946 0)
+      (effects (font (size 1.27 1.27)) (justify left top))
+    )
+    (pin "outRight" output (at 62.865 129.54 0)
+      (effects (font (size 1.27 1.27)) (justify right))
+    )
+    (pin "outLeft" output (at 39.37 137.795 180)
+      (effects (font (size 1.27 1.27)) (justify left))
+    )
+    (pin "outUp" output (at 55.245 143.51 270)
+      (effects (font (size 1.27 1.27)) (justify left))
+    )
+    (pin "outDown" output (at 45.72 124.46 90)
+      (effects (font (size 1.27 1.27)) (justify right))
+    )
+    (instances
+      (project "HierarchyTest"
+        (path "/dc20b726-2806-4869-81d9-be0d53dc7b3c" (page "7"))
       )
     )
@@
     )
   )
+  (sheet (at 78.74 98.425) (size 24.13 17.78) (fields_autoplaced)
+    (stroke (width 0.1524) (type solid))
+    (fill (color 0 0 0 0.0000))
+    (property "Sheetname" "BidirPins" (at 78.74 97.7134 0)
+      (effects (font (size 1.27 1.27)) (justify left bottom))
+    )
+    (property "Sheetfile" "PinsBidir.kicad_sch" (at 78.74 116.7896 0)
+      (effects (font (size 1.27 1.27)) (justify left top))
+    )
+    (pin "biLeft" bidirectional (at 78.74 110.49 180)
+      (effects (font (size 1.27 1.27)) (justify left))
+    )
+    (pin "biDown" bidirectional (at 85.725 98.425 90)
+      (effects (font (size 1.27 1.27)) (justify right))
+    )
+    (pin "biRight" bidirectional (at 102.87 104.14 0)
+      (effects (font (size 1.27 1.27)) (justify right))
+    )
+    (pin "biUp" bidirectional (at 93.345 116.205 270)
+      (effects (font (size 1.27 1.27)) (justify left))
+    )
+    (instances
+      (project "HierarchyTest"
+        (path "/dc20b726-2806-4869-81d9-be0d53dc7b3c" (page "8"))
+      )
+    )
+  )
+  (sheet (at 39.37 98.425) (size 22.86 18.415) (fields_autoplaced)
+    (stroke (width 0.1524) (type solid))
+    (fill (color 0 0 0 0.0000))
+    (property "Sheetname" "InPins" (at 39.37 97.7134 0)
+      (effects (font (size 1.27 1.27)) (justify left bottom))
+    )
+    (property "Sheetfile" "PinsIn.kicad_sch" (at 39.37 117.4246 0)
+      (effects (font (size 1.27 1.27)) (justify left top))
+    )
+    (pin "inDown" input (at 47.625 98.425 90)
+      (effects (font (size 1.27 1.27)) (justify right))
+    )
+    (pin "inLeft" input (at 39.37 111.76 180)
+      (effects (font (size 1.27 1.27)) (justify left))
+    )
+    (pin "inUp" input (at 55.245 116.84 270)
+      (effects (font (size 1.27 1.27)) (justify left))
+    )
+    (pin "inRight" input (at 62.23 104.14 0)
+      (effects (font (size 1.27 1.27)) (justify right))
+    )
+    (instances
+      (project "HierarchyTest"
+        (path "/dc20b726-2806-4869-81d9-be0d53dc7b3c" (page "6"))
+      )
+    )
+  )
   (sheet (at 38.735 75.565) (size 15.24 12.065) (fields_autoplaced)
     (stroke (width 0.1524) (type solid))
@@
     )
   )
+  (sheet (at 58.42 157.48) (size 26.035 19.685) (fields_autoplaced)
+    (stroke (width 0.1524) (type solid))
+    (fill (color 0 0 0 0.0000))
+    (property "Sheetname" "PassivePins" (at 58.42 156.7684 0)
+      (effects (font (size 1.27 1.27)) (justify left bottom))
+    )
+    (property "Sheetfile" "PinsPassive.kicad_sch" (at 58.42 177.7496 0)
+      (effects (font (size 1.27 1.27)) (justify left top))
+    )
+    (pin "passUp" passive (at 76.2 177.165 270)
+      (effects (font (size 1.27 1.27)) (justify left))
+    )
+    (pin "passLeft" passive (at 58.42 170.815 180)
+      (effects (font (size 1.27 1.27)) (justify left))
+    )
+    (pin "passRight" passive (at 84.455 160.655 0)
+      (effects (font (size 1.27 1.27)) (justify right))
+    )
+    (pin "passDown" passive (at 61.595 157.48 90)
+      (effects (font (size 1.27 1.27)) (justify right))
+    )
+    (instances
+      (project "HierarchyTest"
+        (path "/dc20b726-2806-4869-81d9-be0d53dc7b3c" (page "10"))
+      )
+    )
+  )
   (sheet (at 37.465 50.8) (size 18.415 15.875) (fields_autoplaced)
     (stroke (width 0.1524) (type solid))
@@
       )
     )
+  )
+  (sheet (at 79.375 124.46) (size 24.13 19.05) (fields_autoplaced)
+    (stroke (width 0.1524) (type solid))
+    (fill (color 0 0 0 0.0000))
+    (property "Sheetname" "TriPins" (at 79.375 123.7484 0)
+      (effects (font (size 1.27 1.27)) (justify left bottom))
+    )
+    (property "Sheetfile" "PinsTri.kicad_sch" (at 79.375 144.0946 0)
+      (effects (font (size 1.27 1.27)) (justify left top))
+    )
+    (pin "triRight" tri_state (at 103.505 130.175 0)
+      (effects (font (size 1.27 1.27)) (justify right))
+    )
+    (pin "triLeft" tri_state (at 79.375 137.16 180)
+      (effects (font (size 1.27 1.27)) (justify left))
+    )
+    (pin "triUp" tri_state (at 95.885 143.51 270)
+      (effects (font (size 1.27 1.27)) (justify left))
+    )
+    (pin "triDown" tri_state (at 86.995 124.46 90)
+      (effects (font (size 1.27 1.27)) (justify right))
+    )
+    (instances
+      (project "HierarchyTest"
+        (path "/dc20b726-2806-4869-81d9-be0d53dc7b3c" (page "9"))
+      )
+    )
