File: HierarchyTest.kicad_sch (KiCad schematic)
At the start: 3 parts, among them U1 4555, U2 4555, U3 74AHC04

Commit message: aoqifjo
Parts:
- removed unit 2 of U1
- removed U2: 4555, symbol 4xxx_IEEE:4555
- removed U3: 74AHC04, symbol 74xx:74AHC04
Other:
- note added: "New"
