File: accessory.kicad_sch (KiCad schematic)
At the start: 1 part, among them U3 PIC18F13K50-EP

Commit message: updates
Parts:
- renumbered U3 to U7
Changed lines of the file:
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@@
   (symbol (lib_id "MCU_Microchip_PIC18:PIC18F13K50-EP") (at 107.95 64.77 0) (unit 1)
     (in_bom yes) (on_board yes) (dnp no) (fields_autoplaced)
-    (property "Reference" "U3" (at 109.9059 43.815 0)
+    (property "Reference" "U7" (at 109.9059 43.815 0)
       (effects (font (size 1.27 1.27)) (justify left))
     )
@@
       (project "HierarchyTest"
         (path "/dc20b726-2806-4869-81d9-be0d53dc7b3c/f371f224-dc65-4f45-8140-cc26b8de052d/dab23468-3711-408d-b8e3-d53b514e3ccb"
-          (reference "U3") (unit 1)
+          (reference "U7") (unit 1)
+        )
+        (path "/dc20b726-2806-4869-81d9-be0d53dc7b3c/cd9d97e4-da12-4890-a7ea-d84cc7c95661"
+          (reference "U8") (unit 1)
         )
       )
