File: audio.kicad_sch (KiCad schematic)
At the start: 3 parts, among them U2 ${SIM.PARAMS}, U4 ${SIM.PARAMS}, U5 ${SIM.PARAMS}

Commit message: updates
Parts:
- renumbered U5 to U4, U4 to U5, U2 to U6
Changed lines of the file:
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@@
   (symbol (lib_id "Simulation_SPICE:OPAMP") (at 29.21 79.375 180) (unit 1)
     (in_bom yes) (on_board yes) (dnp no) (fields_autoplaced)
-    (property "Reference" "U5" (at 32.3341 70.485 0)
+    (property "Reference" "U4" (at 32.3341 70.485 0)
       (effects (font (size 1.27 1.27)) (justify right))
     )
@@
       (project "HierarchyTest"
         (path "/dc20b726-2806-4869-81d9-be0d53dc7b3c/f371f224-dc65-4f45-8140-cc26b8de052d"
-          (reference "U5") (unit 1)
+          (reference "U4") (unit 1)
         )
       )
@@
   (symbol (lib_id "Simulation_SPICE:OPAMP") (at 98.425 36.195 0) (unit 1)
     (in_bom yes) (on_board yes) (dnp no) (fields_autoplaced)
-    (property "Reference" "U2" (at 121.285 32.7661 0)
+    (property "Reference" "U6" (at 121.285 32.7661 0)
       (effects (font (size 1.27 1.27)))
     )
@@
       (project "HierarchyTest"
         (path "/dc20b726-2806-4869-81d9-be0d53dc7b3c/f371f224-dc65-4f45-8140-cc26b8de052d"
-          (reference "U2") (unit 1)
+          (reference "U6") (unit 1)
         )
       )
@@
   (symbol (lib_id "Simulation_SPICE:OPAMP") (at 70.485 64.135 180) (unit 1)
     (in_bom yes) (on_board yes) (dnp no) (fields_autoplaced)
-    (property "Reference" "U4" (at 73.6091 55.245 0)
+    (property "Reference" "U5" (at 73.6091 55.245 0)
       (effects (font (size 1.27 1.27)) (justify right))
     )
@@
       (project "HierarchyTest"
         (path "/dc20b726-2806-4869-81d9-be0d53dc7b3c/f371f224-dc65-4f45-8140-cc26b8de052d"
-          (reference "U4") (unit 1)
+          (reference "U5") (unit 1)
         )
       )
